File: SolarSpinner_PCB/SolarSpinner.sch (KiCad schematic (older format))
At the start: 21 parts, among them IC1 ATTINY85-P, P1 SOLAR, P10 HOLES, P2 SOLAR_V, P3 MOTOR, P4 ISP, P5 HEADER, P7 LOGO1, P8 LOGO2, Q1 Q_NPN_CBE

Commit message: Updated PCB
Parts:
- removed D2: LED, matts_components:LED-5MM_larg_pad, symbol LED-RESCUE-SolarSpinner
- added D2: LED, REInnovationFootprint:LED-5MM_larg_pad, symbol LED
- IC1: symbol ATTINY85-P -> ATTINY85-P-RESCUE-SolarSpinner
- P4: footprint matts_components:ISP_3x2 -> REInnovationFootprint:ISP_3x2
Connections:
- net GND: now also D2.1 (K)
- net at R6.2: now also D2.2 (A)
Other:
- note added: "ATTiny85 Arduino Pins:\nIC Pin: Arduino Ref:\n1 5/A0/RST\n2 3/A3\n3 4/A2\n4 GND\n5 0 - PWM\n6 1 - PWM\n7 2/A1\n8 +Supply"
Changed lines of the file:
@@
 $EndComp
 $Comp
-L ATTINY85-P IC1
+L ATTINY85-P-RESCUE-SolarSpinner IC1
 U 1 1 58FDDFEF
 P 3600 5150
@@
 F 0 "P4" H 4100 4900 50  0000 C CNN
 F 1 "ISP" H 4100 4500 50  0000 C CNN
-F 2 "matts_components:ISP_3x2" H 4100 3500 50  0001 C CNN
+F 2 "REInnovationFootprint:ISP_3x2" H 4100 3500 50  0001 C CNN
 F 3 "" H 4100 3500 50  0000 C CNN
 	1    4100 4700
@@
 Connection ~ 3150 5650
 $Comp
-L LED-RESCUE-SolarSpinner D2
-U 1 1 5917694E
-P 2150 6000
-F 0 "D2" H 2150 6100 50  0000 C CNN
-F 1 "LED" H 2150 5900 50  0000 C CNN
-F 2 "matts_components:LED-5MM_larg_pad" H 2150 6000 50  0001 C CNN
-F 3 "" H 2150 6000 50  0000 C CNN
-	1    2150 6000
-	0    -1   -1   0
-$EndComp
-$Comp
 L R R6
 U 1 1 591769AF
@@
 L GND #PWR014
 U 1 1 59176BF9
-P 2150 6350
-F 0 "#PWR014" H 2150 6100 50  0001 C CNN
-F 1 "GND" H 2150 6200 50  0000 C CNN
-F 2 "" H 2150 6350 50  0000 C CNN
-F 3 "" H 2150 6350 50  0000 C CNN
-	1    2150 6350
+P 2150 6450
+F 0 "#PWR014" H 2150 6200 50  0001 C CNN
+F 1 "GND" H 2150 6300 50  0000 C CNN
+F 2 "" H 2150 6450 50  0000 C CNN
+F 3 "" H 2150 6450 50  0000 C CNN
+	1    2150 6450
 	1    0    0    -1
 $EndComp
@@
 	2150 5750 2150 5850
 Wire Wire Line
-	2150 6150 2150 6350
+	2150 6250 2150 6450
+Text Notes 1000 5200 0    60   ~ 0
+ATTiny85 Arduino Pins:\nIC Pin:       Arduino Ref:\n1                5/A0/RST\n2                3/A3\n3                4/A2\n4                GND\n5                0 - PWM\n6                1 - PWM\n7                2/A1\n8                +Supply
+$Comp
+L LED D2
+U 1 1 5968E412
+P 2150 6050
+F 0 "D2" H 2150 6150 50  0000 C CNN
+F 1 "LED" H 2150 5950 50  0000 C CNN
+F 2 "REInnovationFootprint:LED-5MM_larg_pad" H 2150 6050 50  0001 C CNN
+F 3 "" H 2150 6050 50  0000 C CNN
+	1    2150 6050
+	0    -1   -1   0
+$EndComp
 $EndSCHEMATC

Commit message: Updated PCB. New Gerber
Parts:
- C1: Supplier 1 (none) -> Aliexpress; Supplier 1 Cost (none) -> 0.4
- C2: Supplier 1 (none) -> Rapid; Supplier 1 Cost (none) -> 0.07
- D1: Supplier 1 (none) -> RS; Supplier 1 Cost (none) -> 0.03
- D2: Description (none) -> 5mm White LED ?; Supplier 1 (none) -> Aliexpress; Supplier 1 Cost (none) -> 0.1
- IC1: Cost 1.12 -> (none); Supplier 1 Cost (none) -> 1.12
- P4: Supplier 1 Cost (none) -> 0.05
- Q1: value Q_NPN_CBE -> BC547
- R1, R2, R3, R4, R5, R6: Supplier 1 Cost (none) -> 0.01
- SC1: Description (none) -> 53x30mm 30mA 5V PV module; Supplier 1 (none) -> Aliexpress; Supplier 1 Cost (none) -> 0.7
Connections:
- net at IC1.5 (PB0(MOSI/DI/SDA/AIN0/OC0A/OC1A/AREF/PCINT0)), P4.4 (P4), P5.6 (P6): now also R6.1
- net at IC1.7 (PB2(SCK/USCK/SCL/T0/INT0/ADC1/PCINT2)), P4.3 (P3), P5.4 (P4): no longer R6.1
Other:
- note added: "ISP Connections:\n1 - MISO\n2 - Vcc\n3 - SCK\n4 - MOSI\n5 - RESET\n6 - GND\n"
