File: SolarSpinner_PCB/SolarSpinner/SolarSpinner.kicad_pcb (KiCad board)
At the start: 2 copper layers, 23 parts, among them IC1 ATTINY85-P, P1 SOLAR, P10 HOLES, P2 SOLAR_V, P3 MOTOR, P4 ISP_3X2, P5 HEADER, P7 LOGO1, P8 LOGO2, Q1 BC547

Commit message: Code Update for different functions
Parts:
- removed P1: SOLAR, REInnovationFootprint:SIL-2_screw_terminal
- removed P10: HOLES, REInnovationFootprint:PCB_Holes_40x50
- removed P8: LOGO2, CuriousElectric3:TCEC_Words_13mm
- added P6: LOGO1, CuriousElectric3:CEC_Globe_10mm_FCU, F.Cu at (89.1, 48.6)
- added R7: 330, REInnovationFootprint:TH_Resistor_1, F.Cu at (142.2, 109.2)
- added R8: 120, REInnovationFootprint:TH_Resistor_1, F.Cu at (142.2, 113.0)
- C2: footprint matts_components:C1_wide_lg_pad -> REInnovationFootprint:C1_wide_lg_pad_2
- D2: value LED -> 1N4001; footprint REInnovationFootprint:LED-5MM_larg_pad -> REInnovationFootprint:TH_Diode_1
- D3: value DIODE -> LED; footprint REInnovationFootprint:TH_Diode_1 -> REInnovationFootprint:LED-5MM_larg_pad
- LS1: value Speaker -> PIEZO
- P2: value SOLAR_V -> ISP_3X2; footprint REInnovationFootprint:SIL-2_LG_PAD -> REInnovationFootprint:ISP_3x2
- P3: value MOTOR -> HEADER; footprint REInnovationFootprint:SIL-2_screw_terminal -> REInnovationFootprint:SIL-7_DIO
- P4: value ISP_3X2 -> MOTOR; footprint REInnovationFootprint:ISP_3x2 -> REInnovationFootprint:SIL-2_screw_terminal
- P5: value HEADER -> HOLES; footprint REInnovationFootprint:SIL-7_DIO -> REInnovationFootprint:PCB_Holes_40x50
- P7: value LOGO1 -> LOGO2; footprint CuriousElectric3:CEC_Globe_10mm_FCU -> CuriousElectric3:TCEC_Words_13mm
- R5: value 330 -> 120
- R6: value 330 -> 100k
- SC1: footprint REInnovationFootprint:PV_50x30mm_round -> REInnovationFootprint:SIL-2_screw_terminal
- moved LS1 118.3 mm to (177.8, 133.3)
- moved SC1 83.0 mm to (162.6, 50.8), turned to 270 degrees
- moved P3 82.2 mm to (80.5, 119.0)
- moved R6 61.2 mm to (142.2, 105.4)
- moved R5 50.2 mm to (142.2, 101.6)
- moved P5 48.8 mm to (119.1, 192.9)
- moved P4 42.0 mm to (217.2, 73.7), turned to 90 degrees
- moved D2 38.6 mm to (166.4, 104.1)
- moved R4 26.7 mm to (142.2, 97.8)
- moved R3 24.3 mm to (142.2, 94.0)
- moved R2 20.9 mm to (142.2, 90.2)
- moved R1 20.7 mm to (142.2, 87.2)
Connections:
- D2 pad 1: GND -> Net-(D2-Pad1)
- D2 pad 2: Net-(D2-Pad2) -> VCC
- D3 pad 1: Net-(D3-Pad1) -> GND
- D3 pad 2: VCC -> Net-(D3-Pad2)
- IC1 pad 5: /LED -> /PIEZO
- IC1 pad 7: /PIEZO -> /LED
- LS1 pad 1: /PIEZO -> Net-(LS1-Pad1)
- P2 pad 1: VCC -> /MOTOR
- P2 pad 2: GND -> VCC
- P3 pad 2: Net-(D3-Pad1) -> /Vsolar
- P4 pad 1: /MOTOR -> VCC
- P4 pad 2: VCC -> Net-(D2-Pad1)
- Q1 pad 1: Net-(D3-Pad1) -> Net-(D2-Pad1)
- R6 pad 1: /LED -> GND
- R6 pad 2: Net-(D2-Pad2) -> Net-(Q1-Pad2)

Commit message: Update of PCB and schematic
Parts:
- D3: footprint REInnovationFootprint:LED-5MM_larg_pad -> REInnovationFootprint:TH_LED-5MM_larg_pad
- LS1: footprint REInnovationFootprint:SIL-2_screw_terminal -> REInnovationFootprint:TH_PIEZO_17x7
- P1: renamed from SC1; value PV_CELL -> PV_IN
- P2: value ISP_3X2 -> ISP
- P3: value HEADER -> IO
- P6: footprint CuriousElectric3:CEC_Globe_10mm_FCU -> CuriousElectric3:2019_011_16_CuriousElectricCompany_Logo_Round_Logo_No_words_KiCAD_10mm_PCBLogo
- R1, R3: value 100k -> 1M
- R2, R4: value 10k -> 100k
- moved P2 122.0 mm to (202.3, 120.0), turned to 90 degrees
- moved P3 109.4 mm to (189.9, 121.5), turned to 0 degrees
- moved P6 108.1 mm to (175.9, 113.0)
- moved C1 87.4 mm to (185.4, 99.3)
- moved P5 82.7 mm to (167.6, 126.0)
- moved IC1 77.2 mm to (198.1, 101.6)
- moved C2 75.2 mm to (199.4, 88.3)
- moved D1 72.2 mm to (179.7, 89.1)
- moved R5 70.7 mm to (212.3, 111.0)
- moved R6 70.5 mm to (212.3, 113.5)
- moved R7 70.4 mm to (212.3, 116.1)
- moved D3 57.9 mm to (209.3, 121.7), turned to 180 degrees
- moved R1 56.6 mm to (195.5, 106.3)
- moved R2 56.5 mm to (195.5, 108.8)
- moved R3 56.1 mm to (195.5, 111.4)
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Other:
- board outline added: 50 x 40 mm
