File: SolarSpinner_PCB/SolarSpinner/SolarSpinner.sch (KiCad schematic (older format))
At the start: 22 parts, among them IC1 ATTINY85-P, P1 SOLAR, P10 HOLES, P3 MOTOR, P4 ISP_3X2, P5 HEADER, P7 LOGO1, P8 LOGO2, Q1 BC547

Commit message: small update
Parts:
- R5: value 330 -> 150
Changed lines of the file:
@@
 LIBS:power
 LIBS:device
-LIBS:transistors
-LIBS:conn
-LIBS:regul
 LIBS:74xx
-LIBS:cmos4000
-LIBS:adc-dac
-LIBS:memory
-LIBS:xilinx
-LIBS:microcontrollers
-LIBS:dsp
-LIBS:microchip
-LIBS:analog_switches
-LIBS:motorola
-LIBS:texas
-LIBS:intel
 LIBS:audio
 LIBS:interface
-LIBS:digital-audio
-LIBS:philips
-LIBS:display
-LIBS:cypress
-LIBS:siliconi
-LIBS:opto
-LIBS:atmel
-LIBS:contrib
-LIBS:valves
 LIBS:SolarSpinner-cache
 EELAYER 29 0
@@
 P 5400 2350
 F 0 "R5" V 5480 2350 50  0000 C CNN
-F 1 "330" V 5400 2350 50  0000 C CNN
+F 1 "150" V 5400 2350 50  0000 C CNN
 F 2 "REInnovationFootprint:TH_Resistor_1" V 5330 2350 50  0001 C CNN
 F 3 "" H 5400 2350 50  0000 C CNN
@@
 Wire Wire Line
 	3100 5600 3400 5600
-$Comp
-L SolarSpinner-rescue:Speaker-Device-SolarSpinner-rescue LS1
-U 1 1 5E8A140A
-P 8700 2050
-F 0 "LS1" H 8870 2046 50  0000 L CNN
-F 1 "Speaker" H 8870 1955 50  0000 L CNN
-F 2 "REInnovationFootprint:SIL-2_screw_terminal" H 8700 1850 50  0001 C CNN
-F 3 "~" H 8690 2000 50  0001 C CNN
-	1    8700 2050
-	1    0    0    -1
-$EndComp
 Text HLabel 2950 5600 0    60   Input ~ 0
 LED
@@
 Text HLabel 7300 1500 0    60   Input ~ 0
 LED
-Text HLabel 8500 1600 0    60   Input ~ 0
-PIEZO
-$Comp
-L matts_components:GND #PWR0101
-U 1 1 5E8C2F6A
-P 8500 2700
-F 0 "#PWR0101" H 8500 2450 50  0001 C CNN
-F 1 "GND" H 8500 2550 50  0000 C CNN
-F 2 "" H 8500 2700 50  0000 C CNN
-F 3 "" H 8500 2700 50  0000 C CNN
-	1    8500 2700
-	1    0    0    -1
-$EndComp
-Wire Wire Line
-	8500 2050 8500 1600
-Wire Wire Line
-	8500 2150 8500 2700
 Wire Wire Line
 	7300 1500 7400 1500
@@
 Wire Wire Line
 	2800 1400 3400 1400
+Wire Wire Line
+	8500 2150 8500 2700
+Wire Wire Line
+	8500 2050 8500 1600
+$Comp
+L matts_components:GND #PWR0101
+U 1 1 5E8C2F6A
+P 8500 2700
+F 0 "#PWR0101" H 8500 2450 50  0001 C CNN
+F 1 "GND" H 8500 2550 50  0000 C CNN
+F 2 "" H 8500 2700 50  0000 C CNN
+F 3 "" H 8500 2700 50  0000 C CNN
+	1    8500 2700
+	1    0    0    -1
+$EndComp
+Text HLabel 8500 1600 0    60   Input ~ 0
+PIEZO
+$Comp
+L SolarSpinner-rescue:Speaker-Device-SolarSpinner-rescue LS1
+U 1 1 5E8A140A
+P 8700 2050
+F 0 "LS1" H 8870 2046 50  0000 L CNN
+F 1 "Speaker" H 8870 1955 50  0000 L CNN
+F 2 "REInnovationFootprint:SIL-2_screw_terminal" H 8700 1850 50  0001 C CNN
+F 3 "~" H 8690 2000 50  0001 C CNN
+	1    8700 2050
+	1    0    0    -1
+$EndComp
 $EndSCHEMATC

Commit message: Code Update for different functions
Parts:
- removed P1: SOLAR, REInnovationFootprint:SIL-2_screw_terminal, symbol SolarSpinner-rescue:Conn_01x02_Female-Connector-SolarSpinner-rescue
- added R6: 100k, REInnovationFootprint:TH_Resistor_1, symbol SolarSpinner-rescue:R-Device-SolarSpinner-rescue
- added R8: 120, REInnovationFootprint:TH_Resistor_1, symbol SolarSpinner-rescue:R-Device-SolarSpinner-rescue
- C2: footprint matts_components:C1_wide_lg_pad -> REInnovationFootprint:C1_wide_lg_pad_2
- D2: renamed from D3; value DIODE -> 1N4001
- LS1: value Speaker -> PIEZO
- R5: value 150 -> 120
- SC1: footprint REInnovationFootprint:PV_50x30mm_round -> REInnovationFootprint:SIL-2_screw_terminal
- renumbered D2 to D3, P4 to P2, P5 to P3, P3 to P4, P10 to P5, P7 to P6, P8 to P7, R6 to R7
Connections:
- net GND: now also R6.1
- net LED: now also IC1.7 (PB2(SCK/USCK/SCL/T0/INT0/ADC1/PCINT2)), P2.3, P3.4 (Pin_4); no longer IC1.5 (PB0(MOSI/DI/SDA/AIN0/OC0A/OC1A/AREF/PCINT0)), P2.4, P3.6 (Pin_6)
- net PIEZO: now also IC1.5 (PB0(MOSI/DI/SDA/AIN0/OC0A/OC1A/AREF/PCINT0)), P2.4, P3.6 (Pin_6), R8.1; no longer IC1.7 (PB2(SCK/USCK/SCL/T0/INT0/ADC1/PCINT2)), LS1.1, P2.3, P3.4 (Pin_4)
- net at Q1.2 (B), R5.2: now also R6.2
- new net: LS1.1, R8.2

Commit message: Update of PCB and schematic
Parts:
- D3: footprint REInnovationFootprint:LED-5MM_larg_pad -> REInnovationFootprint:TH_LED-5MM_larg_pad
- LS1: footprint REInnovationFootprint:SIL-2_screw_terminal -> REInnovationFootprint:TH_PIEZO_17x7
- P1: renamed from SC1; value PV_CELL -> PV_IN
- P2: value ISP_3X2 -> ISP
- P3: value HEADER -> IO
- P6: footprint CuriousElectric3:CEC_Globe_10mm_FCU -> CuriousElectric3:2019_011_16_CuriousElectricCompany_Logo_Round_Logo_No_words_KiCAD_10mm_PCBLogo
- R1, R3: value 100k -> 1M
- R2, R4: value 10k -> 100k
Other:
- moved on the sheet: D2, D3, LS1, P4, Q1, R5, R6, R7, R8
